File: Amp-IRS2092-v2/MultiPSU.sch (EAGLE design)
At the start: 134 parts, among them IC1 ATmega328p, IC2 MID400, IC3 DF10M, K1 ALZ11B12, Q1 7812, Q10 FQA36P15, Q11 FQA36P15, Q12 FQA36P15, Q13 FQA27N25, Q14 FQA27N25, Q15 FQA27N25, Q16 MPSA92, Q17 MPSA42, Q18 MPSA92, Q19 BT169D, Q2 7805, Q20 MPSA92, Q21 MPSA42, Q22 MPSA92, Q23 BC546, Q3 16MHz, Q4 1084-12, Q5 ZVN2106, Q6 ZVN2106, Q7 3LED, Q8 BC546, X1 AC, X10 PROT, X2 RESET, X3 VOL, X4 XFMR_AC, X5 PROT, X6 IR_IN, X7 BIAS, X8 TRI-LED, X9 AC

Commit message: 2024-11-23 21:17
Parts:
- removed D16, D26: 4148, diode:1N4004
- removed D17: 27v, diode:1N4004
- removed Q16, Q20, Q22: MPSA92, transistor-pnp:BC560
- removed Q17, Q21: MPSA42, transistor-npn:BC550B
- added C17: 10uF, resistor:CPOL-EUE3.5-10
- added D15: 4148, diode:1N4004
- added Q24: BC546, transistor-npn:BC550B
- added Q9: BC556, transistor-pnp:BC560
- added R41: 47k, resistor:R-US_0309/10
- added R43: 10k, resistor:R-US_0309/10
- added R46: 10k, resistor:R-US_0411/15
- added R47: 1k1, resistor:R-US_0309/10
- added R56: 4k7, resistor:R-US_0309/10
- added T1, T4, T6: MPSA92, transistor:MPSA92-PNP-TO92-EBC
- added T3, T5: MPSA42, transistor:MPSA42-NPN-TO92-EBC
- Q18: value MPSA92 -> BC556
- R38: value 1k1 -> 330
Connections:
- removed net N$107: D26.A, R38.2, X10-1.S
- removed net N$78 (its old number): Q18.E, X8-1.S
- removed net N$88: Q20.C, R45.1, R50.1
- new net N$108: Q24.C, R56.2
- new net N$109: D15.A, Q18.E, R41.1, R47.2, X10-1.S
- new net N$80: Q9.C, X8-1.S
- new net N$92: C17.+, R45.1, R50.1, T1.E
- new net N$93: Q18.B, R41.2, R56.1
- net AGND: now also C17.-, R43.2; no longer D17.A
- net N$70: now also T5.C; no longer Q17.E
- net N$71: now also T6.C; no longer Q16.E
- net N$72: now also T5.E, T6.E; no longer Q16.C, Q17.C
- net N$73: now also T6.B; no longer Q16.B
- net N$74: now also T5.B; no longer Q17.B
- net N$75: now also Q18.C; no longer D14.C, Q19.E, R37.2, R40.2
- net N$76: now also D14.C, Q19.E, R37.2, R40.2, R47.1
- net N$77: now also Q9.B; no longer Q18.B
- net N$79: now also R38.2, R43.1; no longer D16.C
- net N$81: now also D15.C, Q9.E; no longer D26.C, Q18.C
- net N$89: now also Q24.E, R46.2, T4.C; no longer Q22.E
- net N$90: now also T1.C; no longer Q20.E
- net N$91: now also Q24.B, R46.1; no longer D16.A, D17.C
- net N$94: now also T1.B; no longer Q20.B
- net N$95: now also T3.C; no longer Q21.E
- net N$96: now also T3.E, T4.E; no longer Q21.C, Q22.C
- net N$98: now also T4.B; no longer Q22.B
- net N$99: now also T3.B; no longer Q21.B
Other:
- moved on the sheet: D14, Q18, Q19, R35, R38, R40, R42, R49, X10-1, X10-2, X10-3, X8-1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
