File: Amp-LM1876/Amp-Rev1.sch (EAGLE design)
At the start: 72 parts, among them IC1 LM358N, X1 OUT, X2 IN, X3 IN, X4 AC

Commit message: 2024-11-28 10:20
Parts:
- R30: value 820R -> 820R 1/2w
Changed lines of the file:
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@@
 <part name="D1" library="diode" deviceset="1N4148" device="DO35-7" value="4148"/>
 <part name="C20" library="resistor" deviceset="CPOL-EU" device="E2.5-6" value="1uF"/>
-<part name="R30" library="resistor" deviceset="R-US_" device="0207/10" value="820R"/>
+<part name="R30" library="resistor" deviceset="R-US_" device="0207/10" value="820R 1/2w"/>
 <part name="D2" library="diode" deviceset="1N4148" device="DO35-10" value="5v1"/>
 <part name="GND14" library="supply1" deviceset="GND" device=""/>
